File: hardware/photodiode.sch (KiCad schematic (older format))
At the start: 26 parts

Commit message: added sd_card conponent hardware/sdcard_1051620101.lib connected the sd_card component to the schematic hardware/photodiode.sch generated netlist hardware/photodiode.net
Parts:
- added C8: C, symbol C
- added U3: SC_CARD, symbol SC_CARD
- gave numbers to parts that had none: 26
Connections:
- net labels added: 3v3
- wire segments 54 -> 68
- no-connect marks 1 -> 3
