File: hardware/photodiode.sch (KiCad schematic (older format))
At the start: 26 parts

Commit message: Complete the circuit, make a prototype and an LED blinking firmware
Add the proper PCB footprints for the SD card, crystal oscillator, 3v3 regualtor and user LED
Add connectors for the ADC inputs and serial communication with power port
Create and route the PCB layout
Export the artwork for fabrication. *Inkscape to be used to used for printing svg files plotted*
Add LED blinking firmware for testing the board
Parts:
- removed C?: 0.1uF, symbol C_Small
- removed C? (x2): 18pF, symbol C_Small
- removed CONN?: nokia1202LCD, symbol nokia1202LCD
- removed D?: BAS40-05, symbol BAS40-05
- removed J?: Conn_01x02, symbol Conn_01x02
- removed JP? (x3): Jumper, symbol Jumper_NO_Small
- removed R?: 680, symbol R_Small
- removed R?: 0, symbol R_Small
- removed R?: R_Small, symbol R_Small
- removed Y?: Crystal, symbol Crystal_Small
- added C5: 10nF, Capacitors_SMD:C_0805, symbol C_Small
- added C7: 100n, Capacitors_SMD:C_0805, symbol C
- added J1, J2: Conn_01x04, Pin_Headers:Pin_Header_Angled_1x04_Wide_Pitch2.54mm, symbol Conn_01x04
- added J4: Conn_01x08, photodiode_footprints:Socket_Strip_Straight_1x08_Pitch2.54mm, symbol Conn_01x08
- added MK1, MK2, MK3, MK4: Mounting_Hole, Mounting_Holes:MountingHole_4mm, symbol Mounting_Hole
- added R1: 100, Resistors_SMD:R_1206, symbol R_Small
- added U3: SC_CARD, sdcard:sdcard_1051620101, symbol SC_CARD
- added Y1: Crystal_GND2, CSTGE:CSTCE-G15L, symbol Crystal_GND2
- C1, C2, C3, C4: renamed from C?; footprint (none) -> Capacitors_SMD:C_0805
- C6: renamed from C?; value C_Small -> 100n; footprint (none) -> Capacitors_SMD:C_0805
- D1: renamed from D?; footprint (none) -> LEDs:LED_0805
- J3: renamed from J?; footprint (none) -> photodiode_footprints:Socket_Strip_Straight_1x08_Pitch2.54mm
- P1: renamed from P?; footprint (none) -> Pin_Headers:Pin_Header_Straight_2x05_Pitch1.27mm_SMD
- R2: renamed from R?; value R_Small -> 10k; footprint (none) -> Resistors_SMD:R_1206
- R3: renamed from R?; value R -> 75; footprint (none) -> Resistors_SMD:R_1206
- SW1: renamed from SW?; footprint (none) -> Buttons_Switches_SMD:SW_SPST_EVPBF
- U1: renamed from U?; footprint TO_SOT_Packages_SMD:SOT-223-3_TabPin2 -> TO_SOT_Packages_SMD:SOT-223
- U2: renamed from U?; footprint (none) -> Housings_DFN_QFN:QFN-32-1EP_7x7mm_Pitch0.65mm
Connections:
- net labels added: 3v3, CDET, L_CE, L_CLK, L_LED, L_MOSI, L_RESET
- no-connect marks 1 -> 23
Other:
- note added: "Microcontroller"
- note added: "NOKIA 1616 LCD CONNECTOR"
- note added: "place closest to MCU"
- note removed: "NOKIA 1202 LCD"
